File: PCB/VFD.kicad_pcb (KiCad board)
At the start: 2 copper layers, 247 x 90.9 mm, 78 parts, among them J1 XLR3_Ground, J10 Conn_01x01, J11 Conn_01x01, J2 XLR3_Ground, J3 Conn_01x03_Male, J4 Conn_02x09_Odd_Even, J5 Conn_02x09_Odd_Even, J6 Conn_01x03_Male, J7 Conn_01x01, J8 Conn_01x01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

Commit message: PCB updates
Parts:
- removed R1: 4K7, Resistor_THT:R_Axial_DIN0207_L6.3mm_D2.5mm_P7.62mm_Horizontal
- R15, R16, R17, R18, R19, R20, R21, R22: value R -> 270
- R2: value 4K7 -> 1K
Connections:
- A1 pad 19: /Pot -> /BTN1
- A1 pad 20: /BTN3 -> /BTN2
- A1 pad 21: /BTN2 -> /BTN3
- A1 pad 22: /BTN1 -> /Pot
- J4 pad 10: /BTN2 -> /BTN3
- J4 pad 12: /BTN3 -> /BTN2
- J4 pad 14: /Pot -> /BTN1
- J4 pad 8: /BTN1 -> /Pot
- U1 pad 2: Net-(R1-Pad1) -> GNDA
- U1 pad 3: +5VA -> GNDA
- U1 pad 4: Net-(R1-Pad1) -> GNDA
- U1 pad 6: /DMX- -> /DMX+
- U1 pad 7: /DMX+ -> /DMX-
Routing:
- net Net-(R1-Pad1): track 10.4 -> 0.00 mm
- net GNDA: track 91.1 -> 101.5 mm
- net +5VA: track 32.5 -> 40.1 mm
- net /DMX+: track 9.41 -> 12.6 mm
- net /BTN3: track 33.2 -> 34.5 mm
- net /BTN2: track 34.5 -> 33.2 mm
- net /Pot: track 32.6 -> 33.5 mm, vias 2 -> 4
- net /BTN1: track 33.5 -> 32.6 mm, vias 4 -> 2
- net GNDPWR: vias 10 -> 12
