File: PCB/VFD.kicad_pcb (KiCad board)
At the start: 2 copper layers, 247 x 90.9 mm, 101 parts, among them J1 XLR3_Ground, J10 Conn_01x01, J11 Conn_01x01, J2 XLR3_Ground, J3 Conn_01x03_Male, J4 Conn_02x09_Odd_Even, J5 Conn_02x09_Odd_Even, J6 Conn_01x03_Male, J7 Conn_01x01, J8 Conn_01x01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

Commit message: Updated some component values
Parts:
- R11, R12: value 220k -> 110k
Changed lines of the file:
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@@
-(kicad_pcb (version 20171130) (host pcbnew 5.1.5-52549c5~84~ubuntu18.04.1)
+(kicad_pcb (version 20171130) (host pcbnew 5.1.5-52549c5~86~ubuntu18.04.1)
   (general
     (thickness 1.6)
@@
       (effects (font (size 1 1) (thickness 0.15)))
     )
-    (fp_text value 220k (at 7.62 3.31 90) (layer F.Fab)
+    (fp_text value 110k (at 7.62 3.31 90) (layer F.Fab)
       (effects (font (size 1 1) (thickness 0.15)))
     )
@@
       (effects (font (size 1 1) (thickness 0.15)))
     )
-    (fp_text value 220k (at 7.62 3.31 90) (layer F.Fab)
-      (effects (font (size 1 1) (thickness 0.15)))
-    )
+    (fp_text value 110k (at 7.62 3.31 90) (layer F.Fab)
+      (effects (font (size 1 1) (thickness 0.15)))
+    )
